File: prog.esp8266-01.kicad_pcb (KiCad board)
At the start: 2 copper layers, 36.8 x 29.2 mm, 8 parts, among them J1 SERIAL, J2 Power, SW1 Reset, SW2 PROG, U1 ESP-01v090

Commit message: last version
Variate alcune dimensioni delle piste
Routing:
- net Net-(R3-Pad2): track 78.9 -> 55.0 mm
- net Net-(J1-Pad3): track 41.6 -> 61.9 mm
